File: hardware/CALalarm-r1.sch (EAGLE design)
At the start: 13 parts, among them M1 HAPTIC10MM, Q1 HW5P-1, SW1 ALARM_OFF, T1 2N2222, T2 2N2222, X1 PIEZO

Commit message: squeeze
Other:
- note removed: "Alarm clock based on ESP32 WiFi uController. Synchronizes the time and alarm with Google Calendar."
- moved on the sheet: D1, M1, PCB1P, PCB2+, PCB2P, Q1, R1, R2, R3, R4, T1, T2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
